File: logger.kicad_sch (KiCad schematic)
At the start: 28 parts, among them SW1 BOOT0, U1 STM32U535CBTx, Y1 32.768KHz

Commit message: schematic update
Parts:
- removed R3, R4: 22R, Resistor_SMD:R_0402_1005Metric, symbol Device:R_Small_US
- removed SW1: BOOT0, Button_Switch_SMD:SW_Push_1P1T_NO_Vertical_Wuerth_434133025816, symbol Switch:SW_Push
- removed TP10: PA7, TestPoint:TestPoint_THTPad_D1.0mm_Drill0.5mm, symbol Connector:TestPoint_Small
- removed TP6: PA3, TestPoint:TestPoint_THTPad_D1.0mm_Drill0.5mm, symbol Connector:TestPoint_Small
- removed TP7: PA4, TestPoint:TestPoint_THTPad_D1.0mm_Drill0.5mm, symbol Connector:TestPoint_Small
- removed TP8: PA5, TestPoint:TestPoint_THTPad_D1.0mm_Drill0.5mm, symbol Connector:TestPoint_Small
- removed TP9: PA6, TestPoint:TestPoint_THTPad_D1.0mm_Drill0.5mm, symbol Connector:TestPoint_Small
- added J1: TC2030, Connector:Tag-Connect_TC2030-IDC-NL_2x03_P1.27mm_Vertical, symbol Connector:Conn_ARM_SWD_TagConnect_TC2030-NL
Connections:
- net PA5 is gone; now on net SPI1_SCK: U1.15 (PA5)
- net +3V3: now also J1.1 (VCC)
- net GND: now also J1.5 (GND)
- net SPI1_SCK: no longer U1.39 (PB3)
- net SPI_BARO: now also U1.45 (PB8); no longer U1.38 (PA15)
- net SPI_IMU: now also U1.43 (PB7); no longer U1.42 (PB6)
- net ~{RESET}: now reaches C11.1, U1.7 (NRST)
- net ~{RESET}: now also J1.3 (~{RESET})
- net DEBUG_SWDIO: now reaches U1.34 (PA13)
- net DEBUG_SWDIO: now also J1.2 (SWDIO)
- net PA3: no longer names the net of U1.13 (PA3)
- net PA4: no longer names the net of U1.14 (PA4)
- net PA6: no longer names the net of U1.16 (PA6)
- net PA7: no longer names the net of U1.17 (PA7)
- net SPI_ACCEL renamed DEBUG_SWCLK
- net DEBUG_SWCLK: now also J1.4 (SWCLK)
- net USB_DN: no longer names the net of U1.32 (PA11)
- net USB_DP: no longer names the net of U1.33 (PA12)
- new net DEBUG_SWO: J1.6 (SWO), U1.39 (PB3)
- no-connect marks 13 -> 16
Other:
- sheet Power + USB-C Data renamed Power
- sheet Power ports: added none; removed D+, D-
- sheet SPI1 ports: added none; removed SPI_ACCEL
